Commit message: continue gazebo linking

File: src/jetracer_description/urdf/jetracer.urdf.xacro (robot description, xacro)
@@ -21,4 +21,10 @@
                 <material name="blue"/>
             </visual>
+            <collision>
+                <geometry>
+                    <cylinder radius="${wheel_radius}" length="${wheel_length}"/>
+                </geometry>
+                <origin xyz="0 0 0" rpy="${pi/2.0} 0 0"/>
+            </collision>
             <xacro:cylinder_inertial m="0.3" radius="${wheel_radius}" length="${wheel_length}" o_xyz="0 0 0" o_rpy="${pi/2.0} 0 0"/>
         </link>
@@ -39,4 +45,10 @@
             <material name="green" />
         </visual>
+        <collision>
+            <geometry>
+                <box size="${base_link_length} ${base_link_width} ${base_height}" />
+            </geometry>
+            <origin xyz="0 0 0" rpy="0 0 0" />
+        </collision>
         <xacro:box_inertial m="1.2" x="${base_link_length}" y="${base_link_width}" z="${base_height}" o_xyz="0 0 0" o_rpy="0 0 0"/>
     </link>
@@ -51,7 +63,13 @@
                 <cylinder radius="0.05" length="0.04"/>
             </geometry>
-            <origin xyz="0 0 0" rpy="0 0 0" />
+            <origin xyz="0 0 0" rpy="0 0 0"/>
             <material name="grey" />
         </visual>
+        <collision>
+            <geometry>
+                <cylinder radius="0.05" length="0.04"/>
+            </geometry>
+            <origin xyz="0 0 0" rpy="0 0 0"/>
+        </collision>
         <xacro:cylinder_inertial m="0.1" radius="0.05" length="0.04" o_xyz="0 0 0" o_rpy="0 0 0"/>
     </link>
@@ -64,4 +82,10 @@
 	    <material name="grey"/>
 	  </visual>
+      <collision>
+        <geometry>
+          <box size="0.03 0.03 0.013"/>
+        </geometry>
+         <origin xyz="0 0 0" rpy="0 0 0" />
+      </collision>
       <xacro:box_inertial m="0.1" x="0.03" y="0.03" z="0.013" o_xyz="0 0 0" o_rpy="0 0 0"/>
     </link>

Commit message: add plugins

File: src/jetracer_description/urdf/jetracer.urdf.xacro (robot description, xacro)
@@ -1,6 +1,6 @@
 <?xml version="1.0"?>
 <robot name="jetracer" xmlns:xacro="http://www.ros.org/wiki/xacro">
-    <xacro:property name="base_link_length" value="0.2499"/>
-    <xacro:property name="base_link_width" value="0.1922"/>
+    <xacro:property name="base_length" value="0.2499"/>
+    <xacro:property name="base_width" value="0.1922"/>
     <xacro:property name="base_height" value="0.12"/>
     <xacro:property name="wheel_radius" value="0.0325"/>
@@ -10,5 +10,5 @@
             <parent link="base_link"/>
             <child link="${position}_${side}_wheel"/>
-            <origin xyz="${ base_link_length/3.5 if position=='front' else -0.1 } ${sign * base_link_width * 0.62} -0.06" rpy="0 0 0"/>
+            <origin xyz="${ base_length/3.5 if position=='front' else -0.1 } ${sign * base_width * 0.63} -0.06" rpy="0 0 0"/>
             <axis xyz="0 1 0"/>
         </joint>
@@ -31,4 +31,5 @@
     </xacro:macro>
     <xacro:include filename= "common_properties.xacro"/>
+    <xacro:include filename="jetracer_gazebo.xacro"/>
     <link name="base_footprint"/>
     <joint name="base_joint" type="fixed">
@@ -40,5 +41,5 @@
         <visual>
             <geometry>
-                <box size="${base_link_length} ${base_link_width} ${base_height}" />
+                <box size="${base_length} ${base_width} ${base_height}" />
             </geometry>
             <origin xyz="0 0 0" rpy="0 0 0" />
@@ -47,9 +48,9 @@
         <collision>
             <geometry>
-                <box size="${base_link_length} ${base_link_width} ${base_height}" />
+                <box size="${base_length} ${base_width} ${base_height}" />
             </geometry>
             <origin xyz="0 0 0" rpy="0 0 0" />
         </collision>
-        <xacro:box_inertial m="1.2" x="${base_link_length}" y="${base_link_width}" z="${base_height}" o_xyz="0 0 0" o_rpy="0 0 0"/>
+        <xacro:box_inertial m="1.2" x="${base_length}" y="${base_width}" z="${base_height}" o_xyz="0 0 0" o_rpy="0 0 0"/>
     </link>
     <joint name="base_scan_joint" type="fixed">

Commit message: Lidar and camera plugins added

File: src/jetracer_description/urdf/jetracer.urdf.xacro (robot description, xacro)
@@ -8,4 +8,6 @@
     <xacro:include filename= "common_properties.xacro"/>
     <xacro:include filename="jetracer_gazebo.xacro"/>
+    <xacro:include filename="camera.xacro"/>
+    <xacro:include filename="lidar.xacro"/>
     <xacro:macro name="wheel" params="position side sign">
         <joint name="${position}_${side}_wheel_joint" type="continuous">
@@ -54,46 +56,4 @@
         <xacro:box_inertial m="1.2" x="${base_length}" y="${base_width}" z="${base_height}" o_xyz="0 0 0" o_rpy="0 0 0"/>
     </link>
-    <joint name="base_scan_joint" type="fixed">
-        <parent link="base_link"/>
-        <child link="base_scan"/>
-        <origin xyz="0 0 0.07" rpy="0 0 0"/>
-    </joint>
-    <link name="base_scan">
-        <visual>
-            <geometry>
-                <cylinder r="0.05" l="0.04"/>
-            </geometry>
-            <origin xyz="0 0 0" rpy="0 0 0"/>
-            <material name="grey" />
-        </visual>
-        <collision>
-            <geometry>
-                <cylinder r="0.05" l="0.04"/>
-            </geometry>
-            <origin xyz="0 0 0" rpy="0 0 0"/>
-        </collision>
-        <xacro:cylinder_inertial m="0.1" r="0.05" l="0.04" o_xyz="0 0 0" o_rpy="0 0 0"/>
-    </link>
-    <link name="camera">
-	  <visual>
-	    <geometry>
-	      <box size="0.03 0.03 0.013"/>
-	    </geometry>
-	     <origin xyz="0 0 0" rpy="0 0 0" />
-	    <material name="grey"/>
-	  </visual>
-      <collision>
-        <geometry>
-          <box size="0.03 0.03 0.013"/>
-        </geometry>
-         <origin xyz="0 0 0" rpy="0 0 0" />
-      </collision>
-      <xacro:box_inertial m="0.1" x="0.03" y="0.03" z="0.013" o_xyz="0 0 0" o_rpy="0 0 0"/>
-    </link>
-   <joint name="camera_joint" type="fixed">
-	  <parent link="base_link"/>
-	  <child link="camera"/>
-	  <origin xyz="0.13 0 0.045" rpy="0 0 0"/>
-   </joint>
     <xacro:wheel position="front" side="left" sign="1"/>
     <xacro:wheel position="front" side="right" sign="-1"/>

File: src/jetracer_description/urdf/jetracer_gazebo.xacro (robot description, xacro)
@@ -1,4 +1,12 @@
 <?xml version="1.0"?>
 <robot xmlns:xacro="http://www.ros.org/wiki/xacro">
+    <gazebo reference="front_left_wheel">
+       <mu1 value="0.1"/>
+       <mu2 value="0.1"/>
+    </gazebo>
+    <gazebo reference="front_right_wheel">
+       <mu1 value="0.1"/>
+       <mu2 value="0.1"/>
+    </gazebo>
     <gazebo>
         <plugin
@@ -7,6 +15,6 @@
             <left_joint>base_left_wheel_joint</left_joint>
             <right_joint>base_right_wheel_joint</right_joint>
-            <left_joint>front_left_wheel_joint</left_joint>
-            <right_joint>front_right_wheel_joint</right_joint>
+            <!-- <left_joint>front_left_wheel_joint</left_joint>
+            <right_joint>front_right_wheel_joint</right_joint> -->
             <wheel_seperation>0.4343</wheel_seperation>
             <wheel_radius>0.0325</wheel_radius>
@@ -25,3 +33,10 @@
         </plugin>
     </gazebo>
+    <gazebo>
+        <plugin
+        filename="gz-sim-sensors-system"
+        name="gz::sim::systems::Sensors">
+        <render_engine>ogre2</render_engine>
+        </plugin>
+    </gazebo>
 </robot>
