Commit message: fixed rviz lidar issue with gz_frame_id

File: src/jetracer_description/urdf/jetracer_gazebo.xacro (robot description, xacro)
@@ -35,8 +35,29 @@
     <gazebo>
         <plugin
-        filename="gz-sim-sensors-system"
-        name="gz::sim::systems::Sensors">
-        <render_engine>ogre2</render_engine>
+            filename="gz-sim-sensors-system"
+            name="gz::sim::systems::Sensors">
+            <render_engine>ogre2</render_engine>
         </plugin>
     </gazebo>
+<!-- <gazebo>
+    <plugin
+        filename="gz-sim-triggered-publisher-system"
+        name="gz::sim::systems::TriggeredPublisher">
+        <input type="gz.msgs.Int32" topic="/keyboard/keypress">
+            <match field="data">16777235</match>
+        </input>
+        <output type="gz.msgs.Twist" topic="/cmd_vel">
+            <linear>
+                <x>0.5</x>
+                <y>0.0</y>
+                <z>0.0</z>
+            </linear>
+            <angular>
+                <x>0.0</x>
+                <y>0.0</y>
+                <z>0.0</z>
+            </angular>
+        </output>
+    </plugin>
+</gazebo> -->
 </robot>

File: src/jetracer_description/urdf/lidar.xacro (robot description, xacro)
@@ -1,5 +1,5 @@
 <?xml version="1.0"?>
 <robot xmlns:xacro="http://www.ros.org/wiki/xacro">
-<link name="base_scan">
+    <link name="base_scan">
         <visual>
             <geometry>
@@ -24,5 +24,5 @@
     <gazebo reference="base_scan">
         <sensor name="base_scan" type="gpu_lidar">
-            <pose relative_to='base_scan'>0 0 0 0 0 0</pose>
+            <pose>0 0 0 0 0 0</pose>
             <topic>scan</topic>
             <update_rate>10</update_rate>
@@ -44,11 +44,11 @@
                 <range>
                     <min>0.08</min>
-                    <max>5.0</max>
+                    <max>10</max>
                     <resolution>0.01</resolution>
             </range>
             </ray>
+            <gz_frame_id>base_scan</gz_frame_id>
             <always_on>1</always_on>
             <visualize>true</visualize>
-            <frame_id>base_scan</frame_id>
         </sensor>
     </gazebo>
