Commit message: testing with custom world with slam

File: src/jetracer_description/urdf/camera.xacro (robot description, xacro)
@@ -7,5 +7,5 @@
 	    </geometry>
 	     <origin xyz="0 0 0" rpy="0 0 0" />
-	    <material name="grey"/>
+	    <material name="black"/>
 	  </visual>
       <collision>

File: src/jetracer_description/urdf/common_properties.xacro (robot description, xacro)
@@ -3,4 +3,7 @@
     <material name="grey">
         <color rgba="0.5 0.5 0.5 1" />
+    </material>
+    <material name="black">
+        <color rgba="0.0 0.0 0.0 1.0"/>
     </material>
     <material name="blue">

File: src/jetracer_description/urdf/jetracer.urdf.xacro (robot description, xacro)
@@ -23,5 +23,5 @@
                 </geometry>
                 <origin xyz="0 0 0" rpy="${pi/2.0} 0 0"/>
-                <material name="blue"/>
+                <material name="black"/>
             </visual>
             <collision>

File: src/jetracer_description/urdf/lidar.xacro (robot description, xacro)
@@ -7,5 +7,5 @@
             </geometry>
             <origin xyz="0 0 0" rpy="0 0 0"/>
-            <material name="grey" />
+            <material name="black" />
         </visual>
         <collision>

Commit message: fixed slam map generation and implemented nav2 for navigation

File: src/jetracer_description/urdf/camera.xacro (robot description, xacro)
@@ -2,27 +2,29 @@
 <robot xmlns:xacro="http://www.ros.org/wiki/xacro">
     <link name="camera">
-	  <visual>
-	    <geometry>
-	      <box size="0.03 0.03 0.013"/>
-	    </geometry>
-	     <origin xyz="0 0 0" rpy="0 0 0" />
-	    <material name="black"/>
-	  </visual>
-      <collision>
-        <geometry>
-          <box size="0.03 0.03 0.013"/>
-        </geometry>
-         <origin xyz="0 0 0" rpy="0 0 0" />
-      </collision>
-      <xacro:box_inertial m="0.1" x="0.03" y="0.03" z="0.013" o_xyz="0 0 0" o_rpy="0 0 0"/>
+        <visual>
+            <geometry>
+                <box size="${0.03 * scale} ${0.03 * scale} ${0.013 * scale}"/>
+            </geometry>
+            <origin xyz="0 0 0" rpy="0 0 0" />
+            <material name="black"/>
+        </visual>
+        <collision>
+            <geometry>
+                <box size="${0.03 * scale} ${0.03 * scale} ${0.013 * scale}"/>
+            </geometry>
+            <origin xyz="0 0 0" rpy="0 0 0" />
+        </collision>
+        <!-- Scale mass by scale^3 -->
+        <xacro:box_inertial m="${0.1 * scale * scale * scale}" x="${0.03 * scale}" y="${0.03 * scale}" z="${0.013 * scale}" o_xyz="0 0 0" o_rpy="0 0 0"/>
     </link>
-   <joint name="camera_joint" type="fixed">
-	  <parent link="base_link"/>
-	  <child link="camera"/>
-	  <origin xyz="0.13 0 0.045" rpy="0 0 0"/>
-   </joint>
+    <joint name="camera_joint" type="fixed">
+        <parent link="base_link"/>
+        <child link="camera"/>
+        <!-- Scale xyz positions -->
+        <origin xyz="${0.12 * scale} 0 ${0.015 * scale}" rpy="0 0 0"/>
+    </joint>
     <gazebo reference="camera">
         <sensor name="camera" type="camera">
-            <pose>0.13 0 0.013 0 0 0</pose>
+            <pose>0.12 0 0.015 0 0 0</pose>
                 <topic>camera/image_raw</topic>
                 <update_rate>30</update_rate>

File: src/jetracer_description/urdf/common_properties.xacro (robot description, xacro)
@@ -12,4 +12,28 @@
     <material name="green">
       	<color rgba="0 1 0 1"/>
+    </material>
+    <material name="red">
+        <color rgba="1 0 0 1" />
+    </material>
+    <material name="white">
+        <color rgba="1 1 1 1" />
+    </material>
+    <material name="yellow">
+        <color rgba="1 1 0 1" />
+    </material>
+    <material name="orange">
+        <color rgba="1 0.5 0 1" />
+    </material>
+    <material name="purple">
+        <color rgba="0.5 0 0.5 1" />
+    </material>
+    <material name="pink">
+        <color rgba="1 0.5 0.5 1" />
+    </material>
+    <material name="cyan">
+        <color rgba="0 1 1 1" />
+    </material>
+    <material name="magenta">
+        <color rgba="1 0 1 1" />
     </material>
     <xacro:macro name="box_inertial" params="m x y z o_xyz o_rpy">

File: src/jetracer_description/urdf/jetracer.urdf.xacro (robot description, xacro)
@@ -1,36 +1,82 @@
 <?xml version="1.0"?>
 <robot name="jetracer" xmlns:xacro="http://www.ros.org/wiki/xacro">
-    <xacro:property name="base_length" value="0.2499"/>
-    <xacro:property name="base_width" value="0.1922"/>
-    <xacro:property name="base_height" value="0.12"/>
-    <xacro:property name="wheel_radius" value="0.0325"/>
-    <xacro:property name="wheel_length" value="0.025"/>
+     <xacro:property name="scale" value="3"/>
+     <xacro:property name="wheel_offset_frac" value="0.25"/>
+   <xacro:property name="base_length" value="${0.2499 * scale}"/>
+    <xacro:property name="base_width" value="${0.1922 * scale}"/>
+    <xacro:property name="base_height" value="${0.06 * scale}"/>
+    <xacro:property name="wheel_radius" value="${0.04 * scale}"/>
+    <xacro:property name="wheel_length" value="${0.025 * scale}"/>
     <xacro:include filename= "common_properties.xacro"/>
     <xacro:include filename="jetracer_gazebo.xacro"/>
     <xacro:include filename="camera.xacro"/>
     <xacro:include filename="lidar.xacro"/>
-    <xacro:macro name="wheel" params="position side sign">
-        <joint name="${position}_${side}_wheel_joint" type="continuous">
-            <parent link="base_link" />
-            <child link="${position}_${side}_wheel"/>
-            <origin xyz="${ base_length/3.5 if position=='front' else -0.1 } ${sign * base_width * 0.63} -0.06" rpy="0 0 0"/>
-            <axis xyz="0 1 0"/>
-        </joint>
-        <link name="${position}_${side}_wheel">
-            <visual>
-                <geometry>
-                    <cylinder radius="${wheel_radius}" length="${wheel_length}"/>
-                </geometry>
-                <origin xyz="0 0 0" rpy="${pi/2.0} 0 0"/>
-                <material name="black"/>
-            </visual>
-            <collision>
-                <geometry>
-                    <cylinder radius="${wheel_radius}" length="${wheel_length}"/>
-                </geometry>
-                <origin xyz="0 0 0" rpy="${pi/2.0} 0 0"/>
-            </collision>
-            <xacro:cylinder_inertial m="0.3" r="${wheel_radius}" l="${wheel_length}" o_xyz="0 0 0" o_rpy="${pi/2.0} 0 0"/>
+    <xacro:macro name="steering_wheel" params="position side sign">
+        <xacro:if value="${position=='front'}">
+            <link name="${position}_${side}_steer_link">
+                <xacro:cylinder_inertial m="0.3" r="${wheel_radius}" l="${wheel_length}" o_xyz="0 0 0" o_rpy="${pi/2.0} 0 0"/>
+              </link>
+            <!-- 1) steering joint -->
+            <joint name="${position}_${side}_steer_joint" type="revolute">
+                <parent link="base_link"/>
+                <child  link="${position}_${side}_steer_link"/>
+                <!-- position at same x,y,z as wheel -->
+                <origin xyz="${
+                    base_length/2.4
+                } ${
+                    sign * base_width * 0.63
+                } ${-(base_height*wheel_offset_frac)}" rpy="0 0 0"/>
+                <axis  xyz="0 0 1"/>
+                <limit lower="-0.785" upper="0.785" effort="40" velocity="4"/>
+            </joint>
+            <!-- 2) then the rolling wheel joint, parented to the steer_link -->
+            <joint name="${position}_${side}_wheel_joint" type="continuous">
+                <parent link="${position}_${side}_steer_link"/>
+                <child  link="${position}_${side}_wheel"/>
+                <origin xyz="0 0 0" rpy="0 0 0"/>
+                <axis  xyz="0 1 0"/>
+            </joint>
+            <link name="${position}_${side}_wheel">
+                <visual>
+                    <geometry>
+                        <cylinder radius="${wheel_radius}" length="${wheel_length}"/>
+                    </geometry>
+                    <origin xyz="0 0 0" rpy="${pi/2.0} 0 0"/>
+                    <material name="black"/>
+                </visual>
+                <collision>
+                    <geometry>
+                        <cylinder radius="${wheel_radius}" length="${wheel_length}"/>
+                    </geometry>
+                    <origin xyz="0 0 0" rpy="${pi/2.0} 0 0"/>
+                </collision>
+                <xacro:cylinder_inertial m="0.3" r="${wheel_radius}" l="${wheel_length}" o_xyz="0 0 0" o_rpy="${pi/2.0} 0 0"/>
         </link>
+        </xacro:if>
+        <xacro:if value="${position!='front'}">
+            <!-- rear wheels unchanged -->
+            <joint name="${position}_${side}_wheel_joint" type="continuous">
+                <parent link="base_link"/>
+                <child  link="${position}_${side}_wheel"/>
+                <origin xyz="${-0.1*scale} ${sign * base_width * 0.63} ${-(base_height * wheel_offset_frac)}" rpy="0 0 0"/>
+                <axis xyz="0 1 0"/>
+            </joint>
+            <link name="${position}_${side}_wheel">
+                <visual>
+                    <geometry>
+                        <cylinder radius="${wheel_radius}" length="${wheel_length}"/>
+                    </geometry>
+                    <origin xyz="0 0 0" rpy="${pi/2.0} 0 0"/>
+                    <material name="black"/>
+                </visual>
+                <collision>
+                    <geometry>
+                        <cylinder radius="${wheel_radius}" length="${wheel_length}"/>
+                    </geometry>
+                    <origin xyz="0 0 0" rpy="${pi/2.0} 0 0"/>
+                </collision>
+                <xacro:cylinder_inertial m="0.3" r="${wheel_radius}" l="${wheel_length}" o_xyz="0 0 0" o_rpy="${pi/2.0} 0 0"/>
+            </link>
+        </xacro:if>
     </xacro:macro>
     <link name="base_footprint" />
@@ -38,5 +84,5 @@
         <parent link="base_footprint"/>
         <child link="base_link"/>
-        <origin xyz="0 0 0.0925" rpy="0 0 0"/>
+        <origin xyz="0 0 ${0.05 * scale}" rpy="0 0 0"/>
     </joint>
     <link name="base_link">
@@ -55,8 +101,14 @@
         </collision>
         <xacro:box_inertial m="1.2" x="${base_length}" y="${base_width}" z="${base_height}" o_xyz="0 0 0" o_rpy="0 0 0"/>
+        <sensor name="imu_sensor" type="imu">
+            <always_on>1</always_on>
+            <update_rate>1</update_rate>
+            <visualize>true</visualize>
+            <topic>imu</topic>
+        </sensor>
     </link>
-    <xacro:wheel position="front" side="left" sign="1"/>
-    <xacro:wheel position="front" side="right" sign="-1"/>
-    <xacro:wheel position="base" side="left" sign="1"/>
-    <xacro:wheel position="base" side="right" sign="-1"/>
+    <xacro:steering_wheel position="front" side="left" sign="1"/>
+    <xacro:steering_wheel position="front" side="right" sign="-1"/>
+    <xacro:steering_wheel position="rear" side="left" sign="1"/>
+    <xacro:steering_wheel position="rear" side="right" sign="-1"/>
 </robot>

File: src/jetracer_description/urdf/jetracer_gazebo.xacro (robot description, xacro)
@@ -2,24 +2,10 @@
 <robot xmlns:xacro="http://www.ros.org/wiki/xacro">
     <gazebo reference="front_left_wheel">
-       <mu1 value="0.1"/>
-       <mu2 value="0.1"/>
+       <mu1 value="0.3"/>
+       <mu2 value="0.3"/>
     </gazebo>
     <gazebo reference="front_right_wheel">
-       <mu1 value="0.1"/>
-       <mu2 value="0.1"/>
-    </gazebo>
-    <gazebo>
-        <plugin
-            filename="gz-sim-diff-drive-system"
-            name="gz::sim::systems::DiffDrive">
-            <left_joint>base_left_wheel_joint</left_joint>
-            <right_joint>base_right_wheel_joint</right_joint>
-            <!-- <left_joint>front_left_wheel_joint</left_joint>
-            <right_joint>front_right_wheel_joint</right_joint> -->
-            <wheel_seperation>0.4343</wheel_seperation>
-            <wheel_radius>0.0325</wheel_radius>
-            <frame_id>odom</frame_id>
-            <child_frame_id>base_footprint</child_frame_id>
-        </plugin>
+       <mu1 value="0.3"/>
+       <mu2 value="0.3"/>
     </gazebo>
     <gazebo>
@@ -27,6 +13,8 @@
             filename="gz-sim-joint-state-publisher-system"
             name="gz::sim::systems::JointStatePublisher">
-            <joint_name>base_left_wheel_joint</joint_name>
-            <joint_name>base_right_wheel_joint</joint_name>
+            <joint_name>rear_left_wheel_joint</joint_name>
+            <joint_name>rear_right_wheel_joint</joint_name>
+            <joint_name>front_left_steer_joint</joint_name>
+            <joint_name>front_right_steer_joint</joint_name>
             <joint_name>front_left_wheel_joint</joint_name>
             <joint_name>front_right_wheel_joint</joint_name>
@@ -40,5 +28,35 @@
         </plugin>
     </gazebo>
-<!-- <gazebo>
+    <gazebo>
+        <plugin
+            filename ="gz-sim-imu-system"
+            name="gz::sim::systems::Imu">
+        </plugin>
+    </gazebo>
+    <gazebo>
+        <plugin
+            filename="gz-sim-ackermann-steering-system"
+            name="gz::sim::systems::AckermannSteering">
+            <left_joint>rear_left_wheel_joint</left_joint>
+            <right_joint>rear_right_wheel_joint</right_joint>
+            <left_steering_joint>front_left_steer_joint</left_steering_joint>
+            <right_steering_joint>front_right_steer_joint</right_steering_joint>
+            <ros>
+              <param name="wheel_separation" value="${base_width + 2*wheel_radius}"/>
+              <param name="wheel_radius"     value="${wheel_radius}"/>
+              <param name="steering_limit" value="-0.6"/>
+            </ros>
+            <frame_id>odom</frame_id>
+            <child_frame_id>base_footprint</child_frame_id>
+        </plugin>
+    </gazebo>
+    <gazebo>
+        <plugin
+          filename="gz-sim-keyboard-system"
+          name="gz::sim::systems::Keyboard">
+          <topic>/keyboard/keypress</topic>
+        </plugin>
+      </gazebo>
+<gazebo>
     <plugin
         filename="gz-sim-triggered-publisher-system"
@@ -47,5 +65,5 @@
             <match field="data">16777235</match>
         </input>
-        <output type="gz.msgs.Twist" topic="/cmd_vel">
+        <output type="gz.msgs.Twist" topic="/model/jetracer/cmd_vel">
             <linear>
                 <x>0.5</x>
@@ -60,4 +78,4 @@
         </output>
     </plugin>
-</gazebo> -->
+</gazebo>
 </robot>

File: src/jetracer_description/urdf/lidar.xacro (robot description, xacro)
@@ -4,5 +4,5 @@
         <visual>
             <geometry>
-                <cylinder radius="0.05" length="0.04"/>
+                <cylinder radius="${0.05 * scale}" length="${0.035 * scale}"/>
             </geometry>
             <origin xyz="0 0 0" rpy="0 0 0"/>
@@ -11,18 +11,19 @@
         <collision>
             <geometry>
-                <cylinder radius="0.05" length="0.04"/>
+                <cylinder radius="${0.05 * scale}" length="${0.035 * scale}"/>
             </geometry>
             <origin xyz="0 0 0" rpy="0 0 0"/>
         </collision>
-        <xacro:cylinder_inertial m="0.1" r="0.05" l="0.04" o_xyz="0 0 0" o_rpy="0 0 0"/>
+        <xacro:cylinder_inertial m="${0.1 * scale}" r="${0.05 * scale}" l="${0.035 * scale}" o_xyz="0 0 0" o_rpy="0 0 0"/>
     </link>
-     <joint name="base_scan_joint" type="fixed">
+    <joint name="base_scan_joint" type="fixed">
         <parent link="base_link"/>
         <child link="base_scan"/>
-        <origin xyz="0 0 0.07" rpy="0 0 0"/>
+        <origin xyz="0 0 ${base_height/2.5 + 0.02*scale}" rpy="0 0 0"/>
     </joint>
     <gazebo reference="base_scan">
         <sensor name="base_scan" type="gpu_lidar">
-            <pose>0 0 0 0 0 0</pose>
+            <!-- move up by half the cylinder length (0.04*scale/2 = 0.02*scale) -->
+            <pose relative_to="base_scan">0 0 ${0.025*scale} 0 0 0</pose>
             <topic>scan</topic>
             <update_rate>10</update_rate>
@@ -32,19 +33,13 @@
                         <samples>640</samples>
                         <resolution>1</resolution>
-                        <min_angle>-1.396263</min_angle>
-                        <max_angle>1.396263</max_angle>
+                        <min_angle>-3.14</min_angle>
+                        <max_angle>3.14</max_angle>
                     </horizontal>
-                    <vertical>
-                        <samples>1</samples>
-                        <resolution>0.01</resolution>
-                        <min_angle>0</min_angle>
-                        <max_angle>0</max_angle>
-                    </vertical>
                 </scan>
                 <range>
                     <min>0.08</min>
-                    <max>10</max>
+                    <max>15</max>
                     <resolution>0.01</resolution>
-            </range>
+                </range>
             </ray>
             <gz_frame_id>base_scan</gz_frame_id>
@@ -53,3 +48,3 @@
         </sensor>
     </gazebo>
- </robot>
+</robot>
