Commit message: add inertia link

File: src/jetracer_description/urdf/common_properties.xacro (robot description, xacro)
@@ -10,3 +10,27 @@
       	<color rgba="0 1 0 1"/>
     </material>
+    <xacro:macro name="box_inertial" params="m x y z o_xyz o_rpy">
+        <inertial>
+            <mass value="${m}"/>
+            <origin xyz="${o_xyz}" rpy="${o_rpy}"/>
+            <inertia ixx="${m/12.0*(y*y + z*z)}"
+                     ixy="0"
+                     ixz="0"
+                     iyy="${m/12.0*(x*x + z*z)}"
+                     iyz="0"
+                     izz="${m/12.0*(x*x + y*y)}"/>
+        </inertial>
+    </xacro:macro>
+    <xacro:macro name="cylinder_inertial" params="m radius length o_xyz o_rpy">
+        <inertial>
+            <mass value="${m}"/>
+            <origin xyz="${o_xyz}" rpy="${o_rpy}"/>
+            <inertia ixx="${m/12.0*(3*radius*radius + length*length)}"
+                     ixy="0"
+                     ixz="0"
+                     iyy="${m/12.0*(3*radius*radius + length*length)}"
+                     iyz="0"
+                     izz="${m*radius*radius/2.0}"/>
+        </inertial>
+    </xacro:macro>
 </robot>

File: src/jetracer_description/urdf/jetracer.urdf.xacro (robot description, xacro)
@@ -10,5 +10,5 @@
             <parent link="base_link"/>
             <child link="${position}_${side}_wheel"/>
-            <origin xyz="${ base_link_length/3.5 if position=='front' else -0.1 } ${sign * base_link_width * 0.57} -0.06" rpy="0 0 0"/>
+            <origin xyz="${ base_link_length/3.5 if position=='front' else -0.1 } ${sign * base_link_width * 0.62} -0.06" rpy="0 0 0"/>
             <axis xyz="0 1 0"/>
         </joint>
@@ -21,4 +21,5 @@
                 <material name="blue"/>
             </visual>
+            <xacro:cylinder_inertial m="0.3" radius="${wheel_radius}" length="${wheel_length}" o_xyz="0 0 0" o_rpy="${pi/2.0} 0 0"/>
         </link>
     </xacro:macro>
@@ -38,4 +39,5 @@
             <material name="green" />
         </visual>
+        <xacro:box_inertial m="1.2" x="${base_link_length}" y="${base_link_width}" z="${base_height}" o_xyz="0 0 0" o_rpy="0 0 0"/>
     </link>
     <joint name="base_scan_joint" type="fixed">
@@ -52,4 +54,5 @@
             <material name="grey" />
         </visual>
+        <xacro:cylinder_inertial m="0.1" radius="0.05" length="0.04" o_xyz="0 0 0" o_rpy="0 0 0"/>
     </link>
     <link name="camera">
@@ -61,4 +64,5 @@
 	    <material name="grey"/>
 	  </visual>
+      <xacro:box_inertial m="0.1" x="0.03" y="0.03" z="0.013" o_xyz="0 0 0" o_rpy="0 0 0"/>
     </link>
    <joint name="camera_joint" type="fixed">

Commit message: fixed rviz

File: src/jetracer_description/urdf/common_properties.xacro (robot description, xacro)
@@ -22,14 +22,14 @@
         </inertial>
     </xacro:macro>
-    <xacro:macro name="cylinder_inertial" params="m radius length o_xyz o_rpy">
+    <xacro:macro name="cylinder_inertial" params="m r l o_xyz o_rpy">
         <inertial>
             <mass value="${m}"/>
             <origin xyz="${o_xyz}" rpy="${o_rpy}"/>
-            <inertia ixx="${m/12.0*(3*radius*radius + length*length)}"
+            <inertia ixx="${m/12.0*(3*r*r + l*l)}"
                      ixy="0"
                      ixz="0"
-                     iyy="${m/12.0*(3*radius*radius + length*length)}"
+                     iyy="${m/12.0*(3*r*r + l*l)}"
                      iyz="0"
-                     izz="${m*radius*radius/2.0}"/>
+                     izz="${m*r*r/2.0}"/>
         </inertial>
     </xacro:macro>

File: src/jetracer_description/urdf/jetracer.urdf.xacro (robot description, xacro)
@@ -6,7 +6,9 @@
     <xacro:property name="wheel_radius" value="0.0325"/>
     <xacro:property name="wheel_length" value="0.025"/>
+    <xacro:include filename= "common_properties.xacro"/>
+    <xacro:include filename="jetracer_gazebo.xacro"/>
     <xacro:macro name="wheel" params="position side sign">
         <joint name="${position}_${side}_wheel_joint" type="continuous">
-            <parent link="base_link"/>
+            <parent link="base_link" />
             <child link="${position}_${side}_wheel"/>
             <origin xyz="${ base_length/3.5 if position=='front' else -0.1 } ${sign * base_width * 0.63} -0.06" rpy="0 0 0"/>
@@ -27,34 +29,8 @@
                 <origin xyz="0 0 0" rpy="${pi/2.0} 0 0"/>
             </collision>
-            <xacro:cylinder_inertial m="0.3" radius="${wheel_radius}" length="${wheel_length}" o_xyz="0 0 0" o_rpy="${pi/2.0} 0 0"/>
+            <xacro:cylinder_inertial m="0.3" r="${wheel_radius}" l="${wheel_length}" o_xyz="0 0 0" o_rpy="${pi/2.0} 0 0"/>
         </link>
     </xacro:macro>
-    <xacro:macro name="wheel_link" params="position side sign">
-        <joint name="${position}_${side}_wheel_joint" type="fixed">
-            <parent link="base_link"/>
-            <child link="${position}_${side}_wheel"/>
-            <origin xyz="${ base_length/3.5 if position=='front' else -0.1 } ${sign * base_width * 0.63} -0.06" rpy="0 0 0"/>
-            <axis xyz="0 1 0"/>
-        </joint>
-        <link name="${position}_${side}_wheel">
-            <visual>
-                <geometry>
-                    <cylinder radius="${wheel_radius}" length="${wheel_length}"/>
-                </geometry>
-                <origin xyz="0 0 0" rpy="${pi/2.0} 0 0"/>
-                <material name="blue"/>
-            </visual>
-            <collision>
-                <geometry>
-                    <cylinder radius="${wheel_radius}" length="${wheel_length}"/>
-                </geometry>
-                <origin xyz="0 0 0" rpy="${pi/2.0} 0 0"/>
-            </collision>
-            <xacro:cylinder_inertial m="0.3" radius="${wheel_radius}" length="${wheel_length}" o_xyz="0 0 0" o_rpy="${pi/2.0} 0 0"/>
-        </link>
-    </xacro:macro>
-    <xacro:include filename= "common_properties.xacro"/>
-    <xacro:include filename="jetracer_gazebo.xacro"/>
-    <link name="base_footprint"/>
+    <link name="base_footprint" />
     <joint name="base_joint" type="fixed">
         <parent link="base_footprint"/>
@@ -86,5 +62,5 @@
         <visual>
             <geometry>
-                <cylinder radius="0.05" length="0.04"/>
+                <cylinder r="0.05" l="0.04"/>
             </geometry>
             <origin xyz="0 0 0" rpy="0 0 0"/>
@@ -93,9 +69,9 @@
         <collision>
             <geometry>
-                <cylinder radius="0.05" length="0.04"/>
+                <cylinder r="0.05" l="0.04"/>
             </geometry>
             <origin xyz="0 0 0" rpy="0 0 0"/>
         </collision>
-        <xacro:cylinder_inertial m="0.1" radius="0.05" length="0.04" o_xyz="0 0 0" o_rpy="0 0 0"/>
+        <xacro:cylinder_inertial m="0.1" r="0.05" l="0.04" o_xyz="0 0 0" o_rpy="0 0 0"/>
     </link>
     <link name="camera">

File: src/jetracer_description/urdf/jetracer_gazebo.xacro (robot description, xacro)
@@ -1,18 +1,12 @@
 <?xml version="1.0"?>
 <robot xmlns:xacro="http://www.ros.org/wiki/xacro">
-    <gazebo reference="front_left_wheel">
-        <mu1 value="0.1"/>
-        <mu2 value="0.1"/>
-    </gazebo>
-    <gazebo reference="front_right_wheel">
-        <mu1 value="0.1"/>
-        <mu2 value="0.1"/>
-    </gazebo>
     <gazebo>
         <plugin
-            filename="libignition-gazebo6-diff-drive-system.so"
-            name="ignition::gazebo::systems::DiffDrive">
+            filename="gz-sim-diff-drive-system"
+            name="gz::sim::systems::DiffDrive">
             <left_joint>base_left_wheel_joint</left_joint>
             <right_joint>base_right_wheel_joint</right_joint>
+            <left_joint>front_left_wheel_joint</left_joint>
+            <right_joint>front_right_wheel_joint</right_joint>
             <wheel_seperation>0.4343</wheel_seperation>
             <wheel_radius>0.0325</wheel_radius>
@@ -20,9 +14,13 @@
             <child_frame_id>base_footprint</child_frame_id>
         </plugin>
+    </gazebo>
+    <gazebo>
         <plugin
-            filename="libignition-gazebo6-joint-state-publisher-system.so"
-            name="ignition::gazebo::systems::JointStatePublisher">
+            filename="gz-sim-joint-state-publisher-system"
+            name="gz::sim::systems::JointStatePublisher">
             <joint_name>base_left_wheel_joint</joint_name>
             <joint_name>base_right_wheel_joint</joint_name>
+            <joint_name>front_left_wheel_joint</joint_name>
+            <joint_name>front_right_wheel_joint</joint_name>
         </plugin>
     </gazebo>

Commit message: code-cleanup

File: src/jetracer_description/urdf/common_properties.xacro (robot description, xacro)
@@ -18,22 +18,4 @@
     <material name="white">
         <color rgba="1 1 1 1" />
-    </material>
-    <material name="yellow">
-        <color rgba="1 1 0 1" />
-    </material>
-    <material name="orange">
-        <color rgba="1 0.5 0 1" />
-    </material>
-    <material name="purple">
-        <color rgba="0.5 0 0.5 1" />
-    </material>
-    <material name="pink">
-        <color rgba="1 0.5 0.5 1" />
-    </material>
-    <material name="cyan">
-        <color rgba="0 1 1 1" />
-    </material>
-    <material name="magenta">
-        <color rgba="1 0 1 1" />
     </material>
     <xacro:macro name="box_inertial" params="m x y z o_xyz o_rpy">

File: src/jetracer_description/urdf/jetracer.urdf.xacro (robot description, xacro)
@@ -1,5 +1,5 @@
 <?xml version="1.0"?>
 <robot name="jetracer" xmlns:xacro="http://www.ros.org/wiki/xacro">
-     <xacro:property name="scale" value="3"/>
+     <xacro:property name="scale" value="1.5"/>
      <xacro:property name="wheel_offset_frac" value="0.25"/>
    <xacro:property name="base_length" value="${0.2499 * scale}"/>
@@ -17,9 +17,7 @@
                 <xacro:cylinder_inertial m="0.3" r="${wheel_radius}" l="${wheel_length}" o_xyz="0 0 0" o_rpy="${pi/2.0} 0 0"/>
               </link>
-            <!-- 1) steering joint -->
             <joint name="${position}_${side}_steer_joint" type="revolute">
                 <parent link="base_link"/>
                 <child  link="${position}_${side}_steer_link"/>
-                <!-- position at same x,y,z as wheel -->
                 <origin xyz="${
                     base_length/2.4
@@ -30,5 +28,4 @@
                 <limit lower="-0.785" upper="0.785" effort="40" velocity="4"/>
             </joint>
-            <!-- 2) then the rolling wheel joint, parented to the steer_link -->
             <joint name="${position}_${side}_wheel_joint" type="continuous">
                 <parent link="${position}_${side}_steer_link"/>
@@ -55,5 +52,4 @@
         </xacro:if>
         <xacro:if value="${position!='front'}">
-            <!-- rear wheels unchanged -->
             <joint name="${position}_${side}_wheel_joint" type="continuous">
                 <parent link="base_link"/>
@@ -101,10 +97,4 @@
         </collision>
         <xacro:box_inertial m="1.2" x="${base_length}" y="${base_width}" z="${base_height}" o_xyz="0 0 0" o_rpy="0 0 0"/>
-        <sensor name="imu_sensor" type="imu">
-            <always_on>1</always_on>
-            <update_rate>1</update_rate>
-            <visualize>true</visualize>
-            <topic>imu</topic>
-        </sensor>
     </link>
     <xacro:steering_wheel position="front" side="left" sign="1"/>

File: src/jetracer_description/urdf/lidar.xacro (robot description, xacro)
@@ -24,5 +24,4 @@
     <gazebo reference="base_scan">
         <sensor name="base_scan" type="gpu_lidar">
-            <!-- move up by half the cylinder length (0.04*scale/2 = 0.02*scale) -->
             <pose relative_to="base_scan">0 0 ${0.025*scale} 0 0 0</pose>
             <topic>scan</topic>
